File: a0/a0.kicad_pcb (KiCad board)
At the start: 4 copper layers, 54.6 x 86.3 mm, 132 parts, among them J1 Conn_01x08, J10 Conn_ARM_JTAG_SWD_10, J2 Conn_01x08, J3 Conn_01x08, J4 Conn_01x08, J5 Beagle P8, J6 Beagle P9, J7 ESP32 USB, J8 Screw_Terminal_01x02, J9 BAT_JST_01x02, SW1 SW_Push, SW2 SW_Push, SW5 SMXS-08K-TP, U1 SMXS-02K-TP, U4 ESP32-C6-MINI-1/U, U5 MCP73831-2-OT, U6 XL1509-5.0, U7 AMS1117-3.3, U8 AMS1117-3.3

Commit message: production
Signed-off-by: Rodney Osodo <socials@rodneyosodo.com>
Parts:
- removed G2: LOGO, LOGO
Routing:
- net GND: track 135.6 -> 385.1 mm, vias 63 -> 29
- net USB_D+: track 164.9 -> 81.8 mm, vias 7 -> 4
- net +3V3: track 149.6 -> 175.2 mm, vias 17 -> 4
- net Net-(U7-VI): track 76.5 -> 93.2 mm, vias 10 -> 3
- net FB_5V: track 128.0 -> 143.1 mm, vias 8 -> 1
- net SCK: track 90.8 -> 76.7 mm, vias 8 -> 1
- net GPIO6: track 42.0 -> 28.0 mm, vias 5 -> 2
- net MiBUS1_TX: track 94.1 -> 82.5 mm
- net MiBUS2_TX: track 32.0 -> 22.2 mm, vias 2 -> 0
- net SDA: track 93.4 -> 84.1 mm, vias 11 -> 1
- net MiBUS1_3: track 52.0 -> 61.1 mm, vias 6 -> 1
- net GPIO4: track 42.6 -> 34.2 mm, vias 5 -> 2
- net Net-(U5-STAT): track 5.37 -> 12.5 mm
- net USB_D-: track 88.8 -> 81.7 mm, vias 2 -> 3
- net Net-(U7-VO): track 33.9 -> 40.6 mm, vias 4 -> 0
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