File: a0/expansion.kicad_sch (KiCad schematic)
At the start: 6 parts, among them J1 Conn_01x08, J2 Conn_01x08, J3 Conn_01x08, J4 Conn_01x08, J5 Beagle P8, J6 Beagle P9

Commit message: production
Signed-off-by: Rodney Osodo <socials@rodneyosodo.com>
Parts:
- J1, J2, J3, J4: JLCPCB (none) -> C429957
Changed lines of the file:
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@@
+			)
+		)
+		(property "JLCPCB" "C429957"
+			(at 113.03 144.78 0)
+			(effects
+				(font
+					(size 1.27 1.27)
+				)
+				(hide yes)
 			)
 		)
@@
 			)
 		)
+		(property "JLCPCB" "C429957"
+			(at 110.49 62.23 0)
+			(effects
+				(font
+					(size 1.27 1.27)
+				)
+				(hide yes)
+			)
+		)
 		(pin "8"
 		)
@@
 			)
 		)
+		(property "JLCPCB" "C429957"
+			(at 78.74 144.78 0)
+			(effects
+				(font
+					(size 1.27 1.27)
+				)
+				(hide yes)
+			)
+		)
 		(pin "8"
 		)
@@
 			(at 76.2 62.23 0)
 			(effects
+				(font
+					(size 1.27 1.27)
+				)
+				(hide yes)
+			)
+		)
+		(property "JLCPCB" "C429957"
+			(at 76.2 62.23 0)
+			(effects
