File: modules/E07400M10S/E07400M10S.kicad_pcb (KiCad board)
At the start: 2 copper layers, 25.4 x 28.6 mm, 14 parts, among them J1 Conn_01x08, J2 Conn_01x08, U1 E07-400M10S

Commit message: production
Signed-off-by: Rodney Osodo <socials@rodneyosodo.com>
Routing:
- net GDO0: track 28.3 -> 24.2 mm, vias 0 -> 3
- net GDO1: track 13.3 -> 17.2 mm, vias 0 -> 2
- net SCK: track 20.5 -> 22.0 mm, vias 0 -> 2
- net MISO: track 19.1 -> 20.3 mm
- net CS: track 19.7 -> 20.8 mm, vias 0 -> 2
- net MOSI: track 20.0 -> 21.1 mm, vias 2 -> 3
- net +3V3: track 13.3 -> 13.6 mm, vias 0 -> 2
