File: modules/wmbus/wmbus.kicad_pcb (KiCad board)
At the start: 2 copper layers, 25.4 x 28.6 mm, 15 parts, among them J1 Conn_01x08, J2 Conn_01x08, U2 RC-S2LP-868

Commit message: production
Signed-off-by: Rodney Osodo <socials@rodneyosodo.com>
Routing:
- net SCK: track 10.4 -> 4.49 mm, vias 0 -> 1
- net GND: track 9.64 -> 5.41 mm, vias 10 -> 7
- net CS: track 11.0 -> 8.68 mm, vias 0 -> 1
- net Net-(U2-SDN): track 13.5 -> 14.7 mm
- net MISO: track 5.61 -> 6.51 mm
- net +3V3: track 29.3 -> 28.6 mm
- net MOSI: track 7.49 -> 8.02 mm, vias 0 -> 1
- net SDN: track 24.6 -> 24.4 mm, vias 2 -> 0
