File: modules/sim7080g/sim7080g.kicad_sch (KiCad schematic)
At the start: 42 parts, among them J1 Conn_Coaxial, J2 Conn_01x08, J3 Conn_01x08, J4 Conn_Coaxial, Q1 NPN, Q2 NPN, Q3 NPN, U1 TXB0108RGY, U2 SIM7080G, U3 NANO SIM XG6P H1.35

Commit message: fix: sim7080g module
Signed-off-by: Rodney Osodo <socials@rodneyosodo.com>
Parts:
- removed D2: ESDA6V1SC5, Package_TO_SOT_SMD:SOT-23-5, symbol Power_Protection:ESDA6V1SC5
- removed D3: LED, LED_SMD:LED_0805_2012Metric, symbol Device:LED
- removed J1: Conn_Coaxial, Connector_Coaxial:U.FL_Hirose_U.FL-R-SMT-1_Vertical, symbol Connector:Conn_Coaxial
- removed J3: Conn_01x08, Connector_PinHeader_2.54mm:PinHeader_1x08_P2.54mm_Vertical, symbol Connector_Generic:Conn_01x08
- removed Q1, Q2, Q3: NPN, Package_TO_SOT_SMD:SOT-23, symbol Simulation_SPICE:NPN
- removed U1: TXB0108RGY, Package_DFN_QFN:Texas_RGY_R-PVQFN-N20_EP2.05x3.05mm, symbol Logic_LevelTranslator:TXB0108RGY
- added C14: 1uF, Capacitor_SMD:C_0805_2012Metric, symbol Device:C
- added C15, C16, C17: 100uF, Capacitor_SMD:C_1206_3216Metric, symbol Device:C
- added C18: DNP, Capacitor_SMD:C_0402_1005Metric, symbol Device:C
- added C4: 10uF, Capacitor_SMD:C_0805_2012Metric, symbol Device:C
- added D2: PESD0603V24, Diode_SMD:D_0603_1608Metric, symbol Device:D_TVS
- added D6: ESD9B5.0ST5G, Diode_SMD:D_SOD-923, symbol Diode:ESD9B5.0ST5G
- added D7: LED, LED_SMD:LED_0805_2012Metric, symbol Device:LED
- added D8: ESDA6V1W5, modules:C48677, symbol C48677:ESDA6V1W5
- added FB1: FerriteBead, Inductor_SMD:L_0805_2012Metric, symbol Device:FerriteBead
- added J1: Conn_01x08, Connector_PinHeader_2.54mm:PinHeader_1x08_P2.54mm_Vertical, symbol Connector_Generic:Conn_01x08
- added J3: Conn_Coaxial, Connector_Coaxial:U.FL_Hirose_U.FL-R-SMT-1_Vertical, symbol Connector:Conn_Coaxial
- added L1, L3: DNP, Inductor_SMD:L_0402_1005Metric, symbol Device:L
- added L2: 47nH, Inductor_SMD:L_0402_1005Metric, symbol Device:L
- added Q1, Q2, Q3: MMBT3904, Package_TO_SOT_SMD:SOT-23, symbol Transistor_BJT:MMBT3904
- added R13: 4.7K, Resistor_SMD:R_0805_2012Metric, symbol Device:R
- added R14: 47K, Resistor_SMD:R_0805_2012Metric, symbol Device:R
- added R15: 680, Resistor_SMD:R_0805_2012Metric, symbol Device:R
- added TP1, TP2, TP3, TP4, TP5: TestPoint, TestPoint:TestPoint_Pad_1.0x1.0mm, symbol Connector:TestPoint
- added U1: TXB0108PW, Package_SO:TSSOP-20_4.4x6.5mm_P0.65mm, symbol Logic_LevelTranslator:TXB0108PW
- C10: value 0.1uF -> DNP; JLCPCB C49678 -> C1804; Note (none) -> SIM EMC filter pad - NOT POPULATED. Datasheet Fig.16 shows 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
- C11: value 0.1uF -> 33pF; footprint Capacitor_SMD:C_0805_2012Metric -> Capacitor_SMD:C_0402_1005Metric; JLCPCB C49678 -> C1562
- C12: value 0.1uF -> DNP; footprint Capacitor_SMD:C_0805_2012Metric -> Capacitor_SMD:C_0402_1005Metric; JLCPCB C49678 -> C15008; now left out of the parts list
- C3: value 10uF -> 0.1uF; JLCPCB C15850 -> C49678
- C6: value 22pF -> 0.1uF; JLCPCB C1804 -> C49678
- C7: value 22pF -> DNP; Note (none) -> SIM EMC filter pad - NOT POPULATED. Datasheet Fig.16 shows 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
- C8: value 22pF -> DNP; footprint Capacitor_SMD:C_0805_2012Metric -> Capacitor_SMD:C_0402_1005Metric; JLCPCB C1804 -> C15008; now left out of the parts list
- C9: value 100uF -> DNP; footprint Capacitor_SMD:C_1206_3216Metric -> Capacitor_SMD:C_0805_2012Metric; JLCPCB C15008 -> C1804; Note (none) -> SIM_CLK EMC filter pad - NOT POPULATED. Datasheet Fig.16 sh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
- D4: JLCPCB C6848499 -> C965816
- J4: JLCPCB C88373 -> C88374
- R10: value 47K -> 680; JLCPCB C17713 -> C17798
- R11: value 47K -> 4.7K; JLCPCB C17713 -> C17673
- R12: value 100 -> 47K; JLCPCB C17408 -> C17713
- R2: value 4.7K -> 10K; JLCPCB C17673 -> C17408
- R3: value 22 -> 10; JLCPCB C17561 -> C17415
- R4: value 22 -> 0; footprint Resistor_SMD:R_0805_2012Metric -> Resistor_SMD:R_0402_1005Metric; JLCPCB C17561 -> C17168
- R6: value 47K -> 22; JLCPCB C17713 -> C17561
- R7: value 100 -> 22; JLCPCB C17408 -> C17561
- R9: value 4.7K -> 47K; JLCPCB C17673 -> C17713
Connections:
- net +1V8: now also C2.2, R1.1, R2.2, C4.2, TP5.1, U1.2 (V_{CCA}); no longer C1.2, C3.2
- net +3V3: now also C3.2, R3.2, D6.2 (A2), D7.2 (A), FB1.1, J1.7 (Pin_7), U1.19 (V_{CCB}); no longer C10.1, C11.1, C12.1, C13.1, C2.2, C9.1, J2.7 (Pin_7), R1.1, U2.34 (VBAT), U2.35 (VBAT__1)
- net GND: now also C10.1, C13.1, C8.2, C9.1, R12.2, R9.2, C14.2, C15.2, C16.2, C17.2, C4.1, D2.1 (A1), D6.1 (A1), D8.2, J1.8 (Pin_8), J3.2 (Ext), L1.1, L3.1, Q1.2 (E), Q2.2 (E), Q3.2 (E), R14.1, U1.11 (GND), U1.12 (B8), U1.9 (A8); no longer C10.2, C11.2, C13.2, C8.1, C9.2, R10.2, R11.2, R6.2
- net GNSS_ANT: now also C18.1, L1.2
- net NETLIGHT: now also R13.1; no longer R9.1
- net PWRKEY: now also Q2.3 (C)
- net RF_ANT: now also C8.1, R4.1; no longer J4.1 (In)
- net SIM7080G_CTS: now also J2.2 (Pin_2)
- net SIM7080G_DTR: now also J1.1 (Pin_1), U1.15 (B5); no longer J2.1 (Pin_1)
- net SIM7080G_PWR: now also R11.1, J1.2 (Pin_2); no longer J2.2 (Pin_2), R8.1
- net SIM7080G_RING: now also J2.1 (Pin_1), U1.13 (B7)
- net SIM7080G_RTS: now also J1.3 (Pin_3); no longer J2.3 (Pin_3)
- net SIM7080G_RX: now also J2.4 (Pin_4), U1.18 (B2)
- net SIM7080G_TX: now also J2.3 (Pin_3), U1.20 (B1)
- net SIM_CLK: now also C9.2, R6.1; no longer R4.1
- net SIM_CTS: now also U1.5 (A4)
- net SIM_DATA: now also C10.2, R7.1; no longer R5.1
- net SIM_DTR: now also U1.6 (A5)
- net SIM_RI: now also U1.8 (A7)
- net SIM_RST: now also C7.2, R5.1; no longer R3.1
- net SIM_RTS: now also U1.4 (A3)
- net SIM_RX: now also U1.3 (A2)
- net SIM_TX: now also U1.1 (A1)
- net SIM_VDD: now also C6.2, D8.1; no longer C5.2
- net STATUS: now also R8.1; no longer R2.1
- net at R7.2: now also U3.7 (I/O), D8.5
- net at R8.2: now also R9.1, Q1.1 (B); no longer R11.1
- net at R10.1: now also Q1.3 (C); no longer R9.2
- net at R12.1: now also R11.2, Q2.1 (B)
- net at JP3.1 (A): now also U1.16 (B4)
- net at JP2.1 (A): now also U1.17 (B3)
- net at U2.24 (USB_VBUS): now also TP2.1
- net at U2.25 (USB_DP): now also TP4.1
- net at U2.26 (USB_DM): now also TP3.1
- net SIM_DCD: now reaches U2.5 (UART1_DCD)
- net SIM_DCD: now also U1.7 (A6)
- net at D4.1 (K): now also R10.2; no longer R12.2
- net SIM7080G_DCD: now reaches J2.5 (Pin_5)
- net SIM7080G_DCD: now also U1.14 (B6)
- new net: C1.2, R2.1, TP1.1, U1.10 (OE)
- new net: C12.1, D2.2 (A2), J4.1 (In), R4.2
- new net: C11.2, C18.2, L3.2
- new net: C11.1, J3.1 (In), L2.1
- new net: D8.3, R5.2, U3.2 (RST)
- new net: D8.4, R6.2, U3.3 (CLK)
- new net: Q3.1 (B), R13.2, R14.2
- new net: D7.1 (K), R15.2
- new net: Q3.3 (C), R15.1
- new net VBAT: C13.2, C14.1, C15.1, C16.1, C17.1, FB1.2, U2.34 (VBAT), U2.35 (VBAT__1)
- new net V_ANT: C5.2, L2.2, R3.1
- no-connect marks 38 -> 28
